File: PortableRAM-8MB.kicad_sch (KiCad schematic)
At the start: 37 parts, among them J1 RAM Connector, J2 JTAG_Header_2.54mm_1x06, U1 ATF1502ASL, U11 74HC245, U12 74HC245, U2 AS6C8008-55TIN, U3 AS6C8008-55TIN, U4 AS6C8008-55TIN, U5 AS6C8008-55TIN, U6 AS6C8008-55TIN, U7 AS6C8008-55TIN, U8 AS6C8008-55TIN, U9 AS6C8008-55TIN

Commit message: Add section headers and on-sheet design notes
Seven bold section titles (decode/control, transceivers, low/high
byte arrays, size config, JTAG, connector) and a design-notes block
documenting the memory map, BANKSEL, the WE-split rule, jumper
semantics, CS2, DTACK policy, and the all-5V decision.

Co-Authored-By: Claude Fable 5 <noreply@anthropic.com>
Other:
- note added: "ADDRESS DECODE / CONTROL — ATF1502"
- note added: "BUS TRANSCEIVERS"
- note added: "DESIGN NOTES — v2.0 MEMORY MAP: 4 banks x 2MB (1Mx16 pairs) fill the expansion window 0x100000–0x8FFFFF = 8MB (9MB system total). Banks straddle even-MB boundaries because the window starts at 1MB. BANKSEL (CPLD pin 33) = !A20 — selects which 1MB half of each 2MB bank is active; drives A19 (pin 18) on all SRAMs. Chip A0–A18 = Mac A1–A19. WRITE ENABLES — DO NOT MERGE: /WE (pin 28) = low byte U2–U5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"
- note added: "JTAG"
- note added: "MAC PORTABLE EXPANSION CONNECTOR"
- note added: "MEMORY ARRAY — HIGH BYTE (D8–D15)"
- note added: "MEMORY ARRAY — LOW BYTE (D0–D7)"
- note added: "SIZE CONFIG"
Changed lines of the file:
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@@
+		)
+	)
+	(text "ADDRESS DECODE / CONTROL — ATF1502"
+		(exclude_from_sim no)
+		(at 178 58 0)
+		(effects
+			(font
+				(size 2.54 2.54)
+				(thickness 0.508)
+				(bold yes)
+			)
+			(justify left bottom)
+		)
+	)
+	(text "BUS TRANSCEIVERS"
+		(exclude_from_sim no)
+		(at 272 72 0)
+		(effects
+			(font
+				(size 2.54 2.54)
+				(thickness 0.508)
+				(bold yes)
+			)
+			(justify left bottom)
+		)
+	)
+	(text "MEMORY ARRAY — LOW BYTE (D0–D7)"
+		(exclude_from_sim no)
+		(at 355 42 0)
+		(effects
+			(font
+				(size 2.54 2.54)
+				(thickness 0.508)
+				(bold yes)
+			)
+			(justify left bottom)
+		)
+	)
+	(text "MEMORY ARRAY — HIGH BYTE (D8–D15)"
+		(exclude_from_sim no)
+		(at 355 164 0)
+		(effects
+			(font
+				(size 2.54 2.54)
+				(thickness 0.508)
+				(bold yes)
+			)
+			(justify left bottom)
+		)
+	)
+	(text "SIZE CONFIG"
+		(exclude_from_sim no)
+		(at 196 148 0)
+		(effects
+			(font
+				(size 2.54 2.54)
+				(thickness 0.508)
+				(bold yes)
+			)
+			(justify left bottom)
+		)
+	)
+	(text "JTAG"
+		(exclude_from_sim no)
+		(at 88 150 0)
+		(effects
+			(font
+				(size 2.54 2.54)
+				(thickness 0.508)
+				(bold yes)
+			)
+			(justify left bottom)
+		)
+	)
+	(text "MAC PORTABLE EXPANSION CONNECTOR"
+		(exclude_from_sim no)
+		(at 178 222 0)
+		(effects
+			(font
+				(size 2.54 2.54)
+				(thickness 0.508)
+				(bold yes)
+			)
+			(justify left bottom)
+		)
+	)
+	(text "DESIGN NOTES — v2.0\n\nMEMORY MAP: 4 banks x 2MB (1Mx16 pairs) fill the expansion window\n0x100000–0x8FFFFF = 8MB (9MB system total). Banks straddle even-MB\nboundaries because the window starts at 1MB.\n\nBANKSEL (CPLD pin 33) = !A20 — selects which 1MB half of each 2MB\nbank is active; drives A19 (pin 18) on all SRAMs.\nChip A0–A18 = Mac A1–A19.\n\nWRITE ENABLES — DO NOT MERGE: /WE (pin 28) = low byte U2–U5,\ngated by /LDS. /WEH (pin 30) = high byte U6–U9, gated by /UDS.\nA common WE corrupts the partner byte on 68000 byte writes.\n\nSIZE JUMPER JP1: OPEN = 8MB (all 8 SRAMs). CLOSED = 4MB\n(populate U2, U3, U6, U7 only = banks 0–1). The CPLD never\ndecodes unpopulated space (Mac boot RAM-sizing safety).\n\nCS2 (SRAM pin 40): active-high 2nd enable, tied to +5V (unused).\nDTACK: not driven by this card — the Portable's CPU GLU generates it.\nALL-5V DESIGN: no LDO. AS6C8008 are 2.7–5.5V parts."
+		(exclude_from_sim no)
+		(at 55 240 0)
+		(effects
+			(font
+				(size 1.27 1.27)
+			)
+			(justify left)
 		)
 	)
