File: PortableRAM-8MB.kicad_sch (KiCad schematic)
At the start: 37 parts, among them J1 RAM Connector, J2 JTAG_Header_2.54mm_1x06, U1 ATF1502ASL, U11 74HC245, U12 74HC245, U2 AS6C8008-55TIN, U3 AS6C8008-55TIN, U4 AS6C8008-55TIN, U5 AS6C8008-55TIN, U6 AS6C8008-55TIN, U7 AS6C8008-55TIN, U8 AS6C8008-55TIN, U9 AS6C8008-55TIN

Commit message: Bump to v2.0 — ready to order
Fix SRAM part number AS6C8008-55TIN -> AS6C8008-55ZIN in all 8
schematic instances (ZIN is the current TSOP-II-44 production part).
Bump rev 2.0-dev -> 2.0 in PCB and schematic title blocks.
v0.2 4MB card validated in hardware — gate cleared for v2 order.
Parts:
- U2, U3, U4, U5, U6, U7, U8, U9: value AS6C8008-55TIN -> AS6C8008-55ZIN
Changed lines of the file:
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@@
 	(title_block
 		(title "Mac Portable 4or8MB RAM Card")
-		(date "2026-06-12")
-		(rev "2.0-dev")
+		(date "2026-07-10")
+		(rev "2.0")
 		(company "campbellashe@mac.com")
 		(comment 1 "Designed in North Carolina")
@@
 			)
 		)
-		(property "Value" "AS6C8008-55TIN"
+		(property "Value" "AS6C8008-55ZIN"
 			(at 464.4233 60.96 0)
 			(effects
@@
 			)
 		)
-		(property "Value" "AS6C8008-55TIN"
+		(property "Value" "AS6C8008-55ZIN"
 			(at 356.4733 185.42 0)
 			(effects
@@
 			)
 		)
-		(property "Value" "AS6C8008-55TIN"
+		(property "Value" "AS6C8008-55ZIN"
 			(at 468.2333 185.42 0)
 			(effects
@@
 			)
 		)
-		(property "Value" "AS6C8008-55TIN"
+		(property "Value" "AS6C8008-55ZIN"
 			(at 369.57 59.69 0)
 			(effects
@@
 			)
 		)
-		(property "Value" "AS6C8008-55TIN"
+		(property "Value" "AS6C8008-55ZIN"
 			(at 521.5733 184.15 0)
 			(effects
@@
 			)
 		)
-		(property "Value" "AS6C8008-55TIN"
+		(property "Value" "AS6C8008-55ZIN"
 			(at 413.6233 185.42 0)
 			(effects
@@
 			)
 		)
-		(property "Value" "AS6C8008-55TIN"
+		(property "Value" "AS6C8008-55ZIN"
 			(at 516.4933 62.23 0)
 			(effects
@@
 			)
 		)
-		(property "Value" "AS6C8008-55TIN"
+		(property "Value" "AS6C8008-55ZIN"
 			(at 413.6233 60.96 0)
 			(effects
