File: PortableRAM-8MB.kicad_pcb (KiCad board)
At the start: 4 copper layers, 123 x 81 mm, 38 parts, among them J1 RAM Connector, J2 JTAG_Header_2.54mm_1x06, U1 ATF1502ASL, U11 74HC245, U12 74HC245, U2 AS6C8008-55ZIN, U3 AS6C8008-55TIN, U4 AS6C8008-55TIN, U5 AS6C8008-55TIN, U6 AS6C8008-55TIN, U7 AS6C8008-55TIN, U8 AS6C8008-55TIN, U9 AS6C8008-55TIN

Commit message: Fix AS6C8008-55TIN -> 55ZIN in PCB value fields (7 instances missed earlier)
Parts:
- U3, U4, U5, U6, U7, U8, U9: value AS6C8008-55TIN -> AS6C8008-55ZIN
Changed lines of the file:
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@@
 			)
 		)
-		(property "Value" "AS6C8008-55TIN"
+		(property "Value" "AS6C8008-55ZIN"
 			(at 0 10.16 0)
 			(layer "F.Fab")
@@
 			)
 		)
-		(property "Value" "AS6C8008-55TIN"
+		(property "Value" "AS6C8008-55ZIN"
 			(at 0 10.16 180)
 			(layer "F.Fab")
@@
 			)
 		)
-		(property "Value" "AS6C8008-55TIN"
+		(property "Value" "AS6C8008-55ZIN"
 			(at 0 10.16 180)
 			(layer "F.Fab")
@@
 			)
 		)
-		(property "Value" "AS6C8008-55TIN"
+		(property "Value" "AS6C8008-55ZIN"
 			(at 0 10.16 0)
 			(layer "F.Fab")
@@
 			)
 		)
-		(property "Value" "AS6C8008-55TIN"
+		(property "Value" "AS6C8008-55ZIN"
 			(at 0 10.16 180)
 			(layer "F.Fab")
@@
 			)
 		)
-		(property "Value" "AS6C8008-55TIN"
+		(property "Value" "AS6C8008-55ZIN"
 			(at 0 10.16 0)
 			(layer "F.Fab")
@@
 			)
 		)
-		(property "Value" "AS6C8008-55TIN"
+		(property "Value" "AS6C8008-55ZIN"
 			(at 0 10.16 0)
 			(layer "F.Fab")

Commit message: Add Samtec BCS-125-F-D-HE part number to silkscreen above J1
Other:
- board text added: "Samtec BCS-125-F-D-HE"
Changed lines of the file:
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@@
 	)
 	(embedded_fonts no)
+	(gr_text "Samtec BCS-125-F-D-HE"
+		(at 126 137.5)
+		(layer "F.SilkS")
+		(effects
+			(font
+				(size 1 1)
+				(thickness 0.15)
+			)
+			(justify center)
+		)
+	)
 )
